Commit message: Modify jinyoung urdf

File: jinyoung_description/mr5_v5/urdf/xacro/mr5_gripper_v2.urdf.xacro (robot description, xacro)
@@ -34,4 +34,5 @@
           <mesh filename="package://mr5_v5/urdf/meshes/25BASEPAN.stl" scale="0.001 0.001 0.001"/>
         </geometry>
+        <origin xyz="0 0 0.015" rpy="0 0 0"/>
     </collision>
     <xacro:cylinder_inertial length="0.75" radius="0.5" mass="${base_mass}">
@@ -51,5 +52,6 @@
         </geometry>
         <!--origin xyz="0 -61.835 43.5" rpy="0 0 0"/-->
-        <origin xyz="0.161831 0 -0.01528" rpy="0 1.57 1.57"/>
+        <!--origin xyz="0.161831 0 -0.01528" rpy="0 1.57 1.57"/-->
+        <origin xyz="0.061 0 -0.01528" rpy="0 1.57 1.57"/>
         <material name ="black"/>
       </visual>
@@ -58,4 +60,5 @@
           <mesh filename="package://mr5_v5/urdf/meshes/25_ASM.stl"  scale="0.001 0.001 0.001"/>
         </geometry>
+        <origin xyz="0.061 0 -0.01528" rpy="0 1.57 1.57"/>
     </collision>
     <xacro:cylinder_inertial length="0.6" radius="0.2" mass="${shoulder_mass}">
@@ -76,5 +79,5 @@
           <mesh filename="package://mr5_v5/urdf/meshes/25_ASM.stl"  scale="0.001 0.001 0.001"/>
         </geometry>
-        <origin xyz="0.061831 0 -0.01528" rpy="-1.57 1.57 0"/>
+        <origin xyz="0.061831 0 0.01528" rpy="1.57 -1.57 0"/>
         <material name ="write"/>
       </visual>
@@ -83,4 +86,5 @@
           <mesh filename="package://mr5_v5/urdf/meshes/25_ASM.stl"  scale="0.001 0.001 0.001"/>
         </geometry>
+        <origin xyz="0.061831 0 0.01528" rpy="1.57 -1.57 0"/>
     </collision>
     <xacro:cylinder_inertial length="0.6" radius="0.2" mass="${link1}">
@@ -107,4 +111,5 @@
           <mesh filename="package://mr5_v5/urdf/meshes/25to20.stl"  scale="0.001 0.001 0.001"/>
         </geometry>
+        <origin xyz="0.157935 0 0" rpy="0 0 -1.57"/>
     </collision>
     <xacro:cylinder_inertial length="0.6" radius="0.2" mass="${elbow}">
@@ -131,4 +136,5 @@
           <mesh filename="package://mr5_v5/urdf/meshes/20_ASM.stl"   scale="0.001 0.001 0.001"/>
         </geometry>
+        <origin xyz="0 0 0.0555" rpy="3.14 0 1.57"/>
     </collision>
     <xacro:cylinder_inertial length="0.6" radius="0.2" mass="${link2}">
@@ -148,5 +154,5 @@
           <mesh filename="package://mr5_v5/urdf/meshes/link_elbow.stl"   scale="0.001 0.001 0.001"/>
         </geometry>
-        <origin xyz="-0.054.1 0 0" rpy="-1.57 0 -1.57"/>
+        <origin xyz="-0.0541 0 0" rpy="-1.57 0 -1.57"/>
         <material name ="black"/>
       </visual>
@@ -155,4 +161,5 @@
           <mesh filename="package://mr5_v5/urdf/meshes/link_elbow.stl"   scale="0.001 0.001 0.001"/>
         </geometry>
+        <origin xyz="-0.0541 0 0" rpy="-1.57 0 -1.57"/>
     </collision>
     <xacro:cylinder_inertial length="0.4" radius="0.2" mass="${wrist1}">
@@ -180,4 +187,5 @@
           <mesh filename="package://mr5_v5/urdf/meshes/20to14.stl"   scale="0.001 0.001 0.001"/>
         </geometry>
+        <origin xyz="0.0225 0 0" rpy="0 0 -1.57"/>
     </collision>
     <xacro:cylinder_inertial length="0.6" radius="0.2" mass="${wrist2}">
@@ -204,4 +212,5 @@
           <mesh filename="package://mr5_v5/urdf/meshes/14Series.stl"  scale="0.001 0.001 0.001"/>
         </geometry>
+        <origin xyz="0 0 -0.064" rpy="3.14 0 -1.57"/>
     </collision>
     <xacro:cylinder_inertial length="0.6" radius="0.2" mass="${wrist3}">
@@ -228,4 +237,5 @@
           <mesh filename="package://mr5_v5/urdf/meshes/14Series.stl"  scale="0.001 0.001 0.001"/>
         </geometry>
+        <origin xyz="0 0 -0.06475" rpy="0 3.14 0"/> <!--0 3.14 0-->
     </collision>
     <xacro:cylinder_inertial length="0.6" radius="0.2" mass="1">
@@ -247,5 +257,5 @@
         </geometry>
         <!--origin xyz="0 0 -64.75" rpy="0 3.14 3.14"/-->
-        <origin xyz="0 0 -0.064.75" rpy="0 0 -1.57"/> <!--3.14 0 -1.57 -->
+        <origin xyz="0 0 -0.06475" rpy="3.1415 0 -1.57"/> <!--3.14 0 -1.57 -->
         <material name ="write"/>
       </visual>
@@ -254,4 +264,5 @@
           <mesh filename="package://mr5_v5/urdf/meshes/14Series.stl"  scale="0.001 0.001 0.001"/>
         </geometry>
+        <origin xyz="0 0 -0.06475" rpy="3.1415 0 -1.57"/> <!--3.14 0 -1.57 -->
     </collision>
     <xacro:cylinder_inertial length="0.6" radius="0.2" mass="1">
@@ -279,4 +290,5 @@
         <mesh filename="package://mr5_v5/urdf/meshes/mr14tocamera.stl"  scale="0.001 0.001 0.001"/>
       </geometry>
+      <origin xyz="0 0 0.0125" rpy="3.14 0 1.57"/> <!-- 3.14 0 1.57 -->
   </collision>
     <xacro:cylinder_inertial length="0.6" radius="0.2" mass="1">
@@ -296,5 +308,5 @@
       </geometry>
       <!--origin xyz="0 0 -128.8" rpy="-1.57 3.14 0"/-->
-      <origin xyz="0 0 128.8" rpy="-1.57 0 -1.57"/>
+      <origin xyz="0 0 0.1288" rpy="-1.57 0 -1.57"/>
       <material name ="write"/>
     </visual>
@@ -303,4 +315,5 @@
         <mesh filename="package://mr5_v5/urdf/meshes/parallel_assy_asm.stl"  scale="0.001 0.001 0.001"/>
       </geometry>
+      <origin xyz="0 0 0.1288" rpy="-1.57 0 -1.57"/>
   </collision>
     <xacro:cylinder_inertial length="0.6" radius="0.2" mass="1">
